File: Hardware/Board.brd (EAGLE design)
At the start: 46 x 35 mm, 105 parts, among them IC1 BQ25180YBGR, IC2 DRV2605YZFR, IC3 BMA423_BMA423, IC9 RT6160AWSC, J1 503480-2400, J2 TC2030-IDC_TC2030-IDC, J4 KH-TYPE-C-16P, Q1 20V/4.2A/52mΩ/1.4W, Q3 SI1308EDL-T1-GE3, U1 NORDIC_NRF_4_NRF52840_QF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

Commit message: Manufacturing
Parts:
- moved ANT1 1.39 mm to (6.68, -14.9), turned to 270 degrees
- moved C1 0.82 mm to (4.16, -4.44)
- moved C11 0.49 mm to (3.31, -3.70)
- moved C9 0.42 mm to (3.43, -0.47)
- moved J2 0.29 mm to (-3.92, -6.27)
Routing:
- net GND: track 50.3 -> 48.8 mm, vias 10 -> 35
- net DEC4_6: track 20.8 -> 20.0 mm
- net ALERT: track 80.3 -> 81.1 mm
- net N$3: track 15.3 -> 16.0 mm
- added copper zone on layer 16, net GND
Other:
- board text added: "████████████████████████████████████████████████████████████████████████████████████████ ████████████████████████████████████████████████████████████████████████████████████████ ████████████████████████████████████████████████████████████████████████████████████████ ████████████████████████████████████▒ ░▓██████████████████████████████████ ████████████████████████████████▒ ▒▒░░ ░▒▓███████████████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"

Commit message: Antenna Cutout & Frames
Parts:
- ANT1: value 2450AT18B100E_2450AT18B100E -> 2450AT18B100E
- J2: value TC2030-IDC_TC2030-IDC -> TC2030-IDC
Other:
- outline, holes or cut-outs redrawn
Changed lines of the file:
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@@
 <layer number="14" name="Route14" color="22" fill="1" visible="no" active="no"/>
 <layer number="15" name="Route15" color="23" fill="1" visible="no" active="yes"/>
-<layer number="16" name="Bottom" color="1" fill="1" visible="no" active="yes"/>
+<layer number="16" name="Bottom" color="1" fill="1" visible="yes" active="yes"/>
 <layer number="17" name="Pads" color="2" fill="1" visible="yes" active="yes"/>
 <layer number="18" name="Vias" color="2" fill="1" visible="yes" active="yes"/>
@@
 <layer number="33" name="tFinish" color="6" fill="3" visible="no" active="yes"/>
 <layer number="34" name="bFinish" color="6" fill="6" visible="no" active="yes"/>
-<layer number="35" name="tGlue" color="7" fill="4" visible="yes" active="yes"/>
+<layer number="35" name="tGlue" color="7" fill="4" visible="no" active="yes"/>
 <layer number="36" name="bGlue" color="7" fill="5" visible="no" active="yes"/>
-<layer number="37" name="tTest" color="7" fill="1" visible="yes" active="yes"/>
-<layer number="38" name="bTest" color="7" fill="1" visible="yes" active="yes"/>
-<layer number="39" name="tKeepout" color="4" fill="11" visible="yes" active="yes"/>
+<layer number="37" name="tTest" color="7" fill="1" visible="no" active="yes"/>
+<layer number="38" name="bTest" color="7" fill="1" visible="no" active="yes"/>
+<layer number="39" name="tKeepout" color="4" fill="11" visible="no" active="yes"/>
 <layer number="40" name="bKeepout" color="1" fill="11" visible="no" active="yes"/>
 <layer number="41" name="tRestrict" color="4" fill="10" visible="no" active="yes"/>
@@
 <dimension x1="15.2" y1="-7" x2="15.6" y2="13" x3="20.7" y3="3" textsize="1.778" layer="27" dtype="vertical"/>
 <wire x1="16" y1="-17.5" x2="13.4" y2="-17.5" width="0.1524" layer="20"/>
-<wire x1="8.6" y1="-17.5" x2="2.4" y2="-17.5" width="0.1524" layer="20"/>
 <wire x1="-2.4" y1="-17.5" x2="-8.6" y2="-17.5" width="0.1524" layer="20"/>
 <wire x1="-13.4" y1="-17.5" x2="-16" y2="-17.5" width="0.1524" layer="20"/>
@@
 <wire x1="8.6" y1="-15.7" x2="13.4" y2="-15.7" width="0.1524" layer="20"/>
 <wire x1="-2.4" y1="-15.7" x2="-2.4" y2="-17.5" width="0.1524" layer="20"/>
-<wire x1="2.4" y1="-15.7" x2="2.4" y2="-17.5" width="0.1524" layer="20"/>
-<wire x1="8.6" y1="-15.7" x2="8.6" y2="-17.5" width="0.1524" layer="20"/>
 <wire x1="13.4" y1="-15.7" x2="13.4" y2="-17.5" width="0.1524" layer="20"/>
 <wire x1="-8.6" y1="-15.7" x2="-13.4" y2="-15.7" width="0.1524" layer="20"/>
@@
                      ░░ ░      ░░░░░▒▒▒▒▒▓▓██▓█████████▓█▓█████████████████████████▓▓▒
         ░░░░░▒▒▒▒▒▒▒▓▓▓▓██████████████████████████████████████▓▒▓▓▒▓▓   ░            ░▒ </text>
+<wire x1="8.6" y1="-15.7" x2="8.02" y2="-15.7" width="0.1524" layer="20"/>
+<wire x1="8.02" y1="-15.7" x2="7.73" y2="-15.41" width="0.1524" layer="20"/>
+<wire x1="7.73" y1="-15.41" x2="3.24" y2="-15.41" width="0.1524" layer="20"/>
+<wire x1="3.24" y1="-15.41" x2="2.95" y2="-15.7" width="0.1524" layer="20"/>
+<wire x1="2.95" y1="-15.7" x2="2.4" y2="-15.7" width="0.1524" layer="20"/>
 </plain>
 <attributes>
@@
 </autorouter>
 <elements>
-<element name="ANT1" library="InkTime_v5" library_urn="urn:adsk.wipprod:fs.file:vf.KjXm32SaTAy-5_OOy_6LBw" package="2450AT18B100E_ANTC3216X140N" value="2450AT18B100E_2450AT18B100E" x="6.68" y="-14.92" smashed="yes" rot="R270">
+<element name="ANT1" library="InkTime_v5" library_urn="urn:adsk.wipprod:fs.file:vf.KjXm32SaTAy-5_OOy_6LBw" package="2450AT18B100E_ANTC3216X140N" value="2450AT18B100E" x="6.68" y="-14.92" smashed="yes" rot="R270">
 <attribute name="ARROW_PART_NUMBER" value="2450AT18B100E" x="6.68" y="-14.92" size="1.778" layer="27" rot="R270" display="off"/>
 <attribute name="ARROW_PRICE-STOCK" value="https://www.arrow.com/en/products/2450at18b100e/johanson-dielectrics?utm_currency=USD&amp;region=nac" x="6.68" y="-14.92" size="1.778" layer="27" rot="R270" display="off"/>
@@
 <attribute name="VALUE" x="12.91" y="12.35" size="1.27" layer="27" align="center"/>
 </element>
-<element name="J2" library="InkTime_v5" library_urn="urn:adsk.wipprod:fs.file:vf.KjXm32SaTAy-5_OOy_6LBw" package="TC2030-IDC_TC2030IDC" value="TC2030-IDC_TC2030-IDC" x="-3.92" y="-6.27" smashed="yes" rot="R90">
+<element name="J2" library="InkTime_v5" library_urn="urn:adsk.wipprod:fs.file:vf.KjXm32SaTAy-5_OOy_6LBw" package="TC2030-IDC_TC2030IDC" value="TC2030-IDC" x="-3.92" y="-6.27" smashed="yes" rot="R90">
 <attribute name="ARROW_PART_NUMBER" value="" x="-3.92" y="-6.27" size="1.778" layer="27" rot="R90" display="off"/>
 <attribute name="ARROW_PRICE-STOCK" value="" x="-3.92" y="-6.27" size="1.778" layer="27" rot="R90" display="off"/>
@@
 <wire x1="22.042" y1="8.809" x2="22.05" y2="8.801" width="0.127" layer="16"/>
 <wire x1="22.05" y1="8.801" x2="22.05" y2="6.1" width="0.127" layer="16"/>
-<wire x1="-11.065" y1="-4.895" x2="-10.1" y2="-5.86" width="0.127" layer="16"/>
-<wire x1="-10.1" y1="-5.86" x2="-9.22" y2="-5.86" width="0.127" layer="16"/>
-<wire x1="-9.22" y1="-5.86" x2="-5.835" y2="-2.475" width="0.127" layer="16"/>
+<wire x1="-11.065" y1="-4.895" x2="-10.42" y2="-5.54" width="0.127" layer="16"/>
+<wire x1="-10.42" y1="-5.54" x2="-8.9" y2="-5.54" width="0.127" layer="16"/>
+<wire x1="-8.9" y1="-5.54" x2="-5.835" y2="-2.475" width="0.127" layer="16"/>
 <wire x1="4.48" y1="-1.75" x2="3.76" y2="-1.03" width="0.127" layer="1"/>
 <wire x1="3.76" y1="-1.03" x2="2.902" y2="-1.03" width="0.127" layer="1"/>
@@
 </via>
 <polygon width="0.1524" layer="1" spacing="1.27" pour="solid" thermals="yes">
-<vertex x="8.5568375" y="-15.6354"/>
-<vertex x="8.58484375" y="-15.6238"/>
+<vertex x="-2.4431625" y="-15.6354"/>
+<vertex x="-2.41515625" y="-15.6238"/>
 <vertex x="13.41515625" y="-15.6238"/>
 <vertex x="13.4431625" y="-15.6354"/>
@@
 <vertex x="-2.4762" y="-15.68484375"/>
 <vertex x="-2.4646" y="-15.6568375"/>
-<vertex x="-2.4431625" y="-15.6354"/>
-<vertex x="-2.41515625" y="-15.6238"/>
-<vertex x="2.41515625" y="-15.6238"/>
-<vertex x="2.4431625" y="-15.6354"/>
-<vertex x="2.4646" y="-15.6568375"/>
-<vertex x="2.4762" y="-15.68484375"/>
-<vertex x="2.4762" y="-17.4238"/>
-<vertex x="8.5238" y="-17.4238"/>
-<vertex x="8.5238" y="-15.68484375"/>
-<vertex x="8.5354" y="-15.6568375"/>
 </polygon>
 <wire x1="21.585" y1="10.2" x2="20.61" y2="10.2" width="0.15" layer="1"/>
@@
 <wire x1="7.41" y1="-1.6" x2="7.13" y2="-1.6" width="0.127" layer="1"/>
 <polygon width="0.1524" layer="16" spacing="1.27" pour="solid" thermals="yes">
-<vertex x="-15.9354" y="-6.9431625"/>
-<vertex x="-15.9568375" y="-6.9646"/>
-<vertex x="-15.98484375" y="-6.9762"/>
-<vertex x="-22.9238" y="-6.9762"/>
-<vertex x="-22.9238" y="-10.49784375"/>
-<vertex x="-22.880140625" y="-11.27521875"/>
-<vertex x="-22.7500875" y="-12.040675"/>
-<vertex x="-22.53514375" y="-12.786753125"/>
-<vertex x="-22.23801875" y="-13.504078125"/>
-<vertex x="-21.862440625" y="-14.183628125"/>
-<vertex x="-21.413159375" y="-14.816834375"/>
-<vertex x="-20.895778125" y="-15.395778125"/>
-<vertex x="-20.316834375" y="-15.913159375"/>
-<vertex x="-19.683628125" y="-16.362440625"/>
-<vertex x="-19.004078125" y="-16.73801875"/>
-<vertex x="-18.286753125" y="-17.03514375"/>
-<vertex x="-17.540675" y="-17.2500875"/>
-<vertex x="-16.77521875" y="-17.380140625"/>
-<vertex x="-15.99784375" y="-17.4238"/>
-<vertex x="-13.4762" y="-17.4238"/>
-<vertex x="-13.4762" y="-15.68484375"/>
-<vertex x="-13.4646" y="-15.6568375"/>
-<vertex x="-13.4431625" y="-15.6354"/>
-<vertex x="-13.41515625" y="-15.6238"/>
-<vertex x="-8.58484375" y="-15.6238"/>
-<vertex x="-8.5568375" y="-15.6354"/>
-<vertex x="-8.5354" y="-15.6568375"/>
-<vertex x="-8.5238" y="-15.68484375"/>
-<vertex x="-8.5238" y="-17.4238"/>
-<vertex x="-2.4762" y="-17.4238"/>
-<vertex x="-2.4762" y="-15.68484375"/>
-<vertex x="-2.4646" y="-15.6568375"/>
 <vertex x="-2.4431625" y="-15.6354"/>
 <vertex x="-2.41515625" y="-15.6238"/>
-<vertex x="2.41515625" y="-15.6238"/>
-<vertex x="2.4431625" y="-15.6354"/>
-<vertex x="2.4646" y="-15.6568375"/>
-<vertex x="2.4762" y="-15.68484375"/>
-<vertex x="2.4762" y="-17.4238"/>
-<vertex x="8.5238" y="-17.4238"/>
-<vertex x="8.5238" y="-15.68484375"/>
-<vertex x="8.5354" y="-15.6568375"/>
-<vertex x="8.5568375" y="-15.6354"/>
-<vertex x="8.58484375" y="-15.6238"/>
 <vertex x="13.41515625" y="-15.6238"/>
 <vertex x="13.4431625" y="-15.6354"/>
@@
 <vertex x="-15.9238" y="6.91515625"/>
 <vertex x="-15.9238" y="-6.91515625"/>
+<vertex x="-15.9354" y="-6.9431625"/>
+<vertex x="-15.9568375" y="-6.9646"/>
+<vertex x="-15.98484375" y="-6.9762"/>
+<vertex x="-22.9238" y="-6.9762"/>
+<vertex x="-22.9238" y="-10.49784375"/>
+<vertex x="-22.880140625" y="-11.27521875"/>
+<vertex x="-22.7500875" y="-12.040675"/>
+<vertex x="-22.53514375" y="-12.786753125"/>
+<vertex x="-22.23801875" y="-13.504078125"/>
+<vertex x="-21.862440625" y="-14.183628125"/>
+<vertex x="-21.413159375" y="-14.816834375"/>
+<vertex x="-20.895778125" y="-15.395778125"/>
+<vertex x="-20.316834375" y="-15.913159375"/>
+<vertex x="-19.683628125" y="-16.362440625"/>
+<vertex x="-19.004078125" y="-16.73801875"/>
+<vertex x="-18.286753125" y="-17.03514375"/>
+<vertex x="-17.540675" y="-17.2500875"/>
+<vertex x="-16.77521875" y="-17.380140625"/>
+<vertex x="-15.99784375" y="-17.4238"/>
+<vertex x="-13.4762" y="-17.4238"/>
+<vertex x="-13.4762" y="-15.68484375"/>
+<vertex x="-13.4646" y="-15.6568375"/>
+<vertex x="-13.4431625" y="-15.6354"/>
+<vertex x="-13.41515625" y="-15.6238"/>
+<vertex x="-8.58484375" y="-15.6238"/>
+<vertex x="-8.5568375" y="-15.6354"/>
+<vertex x="-8.5354" y="-15.6568375"/>
+<vertex x="-8.5238" y="-15.68484375"/>
+<vertex x="-8.5238" y="-17.4238"/>
+<vertex x="-2.4762" y="-17.4238"/>
+<vertex x="-2.4762" y="-15.68484375"/>
+<vertex x="-2.4646" y="-15.6568375"/>
 </polygon>
 <via x="4.56" y="-11.54" extent="1-16" drill="0.35" alwaysstop="yes">
