File: Hardware/Schematic.sch (EAGLE design)
At the start: 105 parts, among them IC1 BQ25180YBGR, IC2 DRV2605YZFR, IC3 BMA423_BMA423, IC9 RT6160AWSC, J1 503480-2400, J2 TC2030-IDC_TC2030-IDC, J4 KH-TYPE-C-16P, Q1 20V/4.2A/52mΩ/1.4W, Q3 SI1308EDL-T1-GE3, U1 NORDIC_NRF_4_NRF52840_QF, U3 MAX17048G+T10, X1 32MHz, X2 32.768kHz

Commit message: Antenna Cutout & Frames
Parts:
- ANT1: value 2450AT18B100E_2450AT18B100E -> 2450AT18B100E
- J2: value TC2030-IDC_TC2030-IDC -> TC2030-IDC
Other:
- moved on the sheet: C19, C23, C24, C25, C33, C37, C38, C39, C42, C43, EPD_C1, EPD_C10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
